File: PCB/TitanBoard V1.kicad_pcb (KiCad board)
At the start: 2 copper layers, 411.8 x 121 mm, 212 parts, among them J1 OLED_128x32, U1 Raspberry_Pi_Pico

Commit message: updated footprints
made space for the plate mounted stabilizers
Parts:
- moved D92 15.1 mm to (820.2, 47.2), turned to 0 degrees
- moved D93 14.5 mm to (820.8, 66.2), turned to 0 degrees
- moved D94 14.5 mm to (820.8, 85.3), turned to 0 degrees
- moved D95 14.5 mm to (820.8, 104.3), turned to 0 degrees
Routing:
- net COL4: track 682.8 -> 713.4 mm
- net COL6: track 547.6 -> 569.0 mm
- net COL13: track 465.8 -> 484.9 mm
- net Net-(D70-A): track 17.3 -> 35.3 mm
- net Net-(S36-Pad1): track 311.5 -> 327.8 mm
- net Net-(D100-A): track 57.7 -> 72.5 mm
- net ROW5: track 365.8 -> 376.2 mm
- net ROW1: track 298.2 -> 308.2 mm
- net ROW3: track 333.7 -> 342.8 mm
- net Net-(D95-A): track 7.73 -> 15.8 mm
- net Net-(D94-A): track 7.73 -> 15.8 mm
- net Net-(D93-A): track 7.73 -> 15.8 mm
- net Net-(D92-A): track 7.73 -> 15.5 mm
- net Net-(D5-A): track 19.6 -> 25.9 mm
- net COL11: track 583.8 -> 589.7 mm
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